File: board/spark.kicad_pcb (KiCad board)
At the start: 4 copper layers, 198 x 85 mm, 58 parts, among them J1 RJ45, J2 RJ45, P5 Raspberry_Pi_2_3, Q1 AO3400A, Q2 AO3400A, Q22 AO3400A, Q3 AO3400A, Q4 AO3400A, Q5 AO3400A, Q6 AO3400A, U1 PCA9544APW, U11 MAX11614, U2 PCA9306DC1, U3 LD1117S18TR_SOT223, U4 LD1117S25TR_SOT223, U5 LD1117S33TR_SOT223, U6 LD1117S12TR_SOT223, U7 TCA9535DBR, U8 TXB0104RUT

Commit message: feat: breaking up longer traces
Routing:
- net +5V: track 25.5 -> 26.2 mm, vias 13 -> 14
- net SCL 0: vias 2 -> 4
- net SDA 0: vias 2 -> 4
Changed lines of the file:
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@@
+	)
+	(segment
+		(start 73.05 83)
+		(end 71.25 83)
+		(width 0.8)
+		(layer "F.Cu")
+		(net 2)
 	)
 	(segment
@@
 	)
 	(segment
-		(start 73.05 83)
-		(end 72 83)
-		(width 0.8)
-		(layer "F.Cu")
-		(net 2)
-	)
-	(segment
 		(start 48.35 49.8)
 		(end 47.2 49.8)
@@
 		(size 0.6)
 		(drill 0.4)
+		(layers "F.Cu" "B.Cu")
+		(net 2)
+	)
+	(via
+		(at 71.25 83)
+		(size 0.5)
+		(drill 0.3)
 		(layers "F.Cu" "B.Cu")
 		(net 2)
@@
 		(net 25)
 	)
-	(via
-		(at 88 125.5)
-		(size 0.6)
-		(drill 0.4)
-		(layers "F.Cu" "B.Cu")
+	(segment
+		(start 88 125.5)
+		(end 87.875 125.375)
+		(width 0.254)
+		(layer "F.Cu")
 		(net 25)
 	)
-	(segment
-		(start 88 125.5)
-		(end 78.5 116)
+	(via
+		(at 87.875 125.375)
+		(size 0.6)
+		(drill 0.4)
+		(layers "F.Cu" "B.Cu")
+		(net 25)
+	)
+	(segment
+		(start 56.92 116)
+		(end 20.77 79.85)
 		(width 0.254)
 		(layer "B.Cu")
@@
 	)
 	(segment
-		(start 56.92 116)
-		(end 20.77 79.85)
+		(start 78.5 116)
+		(end 56.92 116)
 		(width 0.254)
 		(layer "B.Cu")
@@
 	)
 	(segment
-		(start 78.5 116)
-		(end 56.92 116)
+		(start 87.875 125.375)
+		(end 78.5 116)
 		(width 0.254)
 		(layer "B.Cu")
@@
 	)
 	(segment
+		(start 62.947341 86.802657)
+		(end 54.822342 78.677658)
+		(width 0.254)
+		(layer "F.Cu")
+		(net 72)
+	)
+	(segment
 		(start 28.175 48.685)
 		(end 28.175 50.1375)
@@
 		(net 72)
 	)
+	(segment
+		(start 62.947341 86.802659)
+		(end 62.947341 86.802657)
+		(width 0.254)
+		(layer "F.Cu")
+		(net 72)
+	)
+	(via
+		(at 54.822342 78.677658)
+		(size 0.6)
+		(drill 0.4)
+		(layers "F.Cu" "B.Cu")
+		(net 72)
+	)
+	(via
+		(at 62.947341 86.802659)
+		(size 0.6)
+		(drill 0.4)
+		(layers "F.Cu" "B.Cu")
+		(net 72)
+	)
 	(via
 		(at 28 51.25)
@@
 		(drill 0.4)
 		(layers "F.Cu" "B.Cu")
+		(net 72)
+	)
+	(segment
+		(start 62.947342 86.802659)
+		(end 84.825001 108.680318)
+		(width 0.254)
+		(layer "In2.Cu")
 		(net 72)
 	)
@@
 	)
 	(segment
+		(start 54.822341 78.677658)
+		(end 54.822342 78.677658)
+		(width 0.254)
+		(layer "In2.Cu")
+		(net 72)
+	)
+	(segment
+		(start 62.947341 86.802659)
+		(end 62.947342 86.802659)
+		(width 0.254)
+		(layer "In2.Cu")
+		(net 72)
+	)
+	(segment
 		(start 28 51.855317)
-		(end 84.825001 108.680318)
+		(end 54.822341 78.677658)
 		(width 0.254)
 		(layer "In2.Cu")
 		(net 72)
+	)
+	(segment
+		(start 53.729918 79.520082)
+		(end 61.854918 87.645082)
+		(width 0.254)
+		(layer "F.Cu")
+		(net 73)
 	)
 	(segment
@@
 	)
 	(via
+		(at 53.729918 79.520082)
+		(size 0.6)
+		(drill 0.4)
+		(layers "F.Cu" "B.Cu")
+		(net 73)
+	)
+	(via
 		(at 86.761583 110.767163)
+		(size 0.6)
+		(drill 0.4)
+		(layers "F.Cu" "B.Cu")
+		(net 73)
+	)
+	(via
+		(at 61.854918 87.645082)
 		(size 0.6)
 		(drill 0.4)
@@
 	(segment
 		(start 27.423 53.213164)
-		(end 84.959836 110.75)
+		(end 53.729918 79.520082)
 		(width 0.254)
 		(layer "In2.Cu")
@@
 		(width 0.254)
 		(layer "In2.Cu")
+		(net 73)
+	)
+	(segment
+		(start 61.854918 87.645082)
+		(end 84.959836 110.75)
+		(width 0.254)
+		(layer "In2.Cu")

Commit message: feat: rev 2
Parts:
- removed D16, D17: Active LED, LED_SMD:LED_0402_1005Metric
- removed Q1, Q2, Q22, Q3, Q4, Q5, Q6: AO3400A, Package_TO_SOT_SMD:SOT-23
- removed R22, R23, R24, R25, R26, R27, R28, R29, R30, R31, R32, R33: 4.7k, Resistor_SMD:R_0402_1005Metric
- removed the R3 at (77.0, 70.1)
- removed the R4 at (77.0, 77.0)
- removed the R5 at (77.0, 82.5)
- removed the R6 at (81.5, 111.0)
- removed the R7 at (87.0, 113.5)
- removed U1: PCA9544APW, Package_SO:TSSOP-20_4.4x6.5mm_P0.65mm
- removed U11: MAX11614, Package_SO:QSOP-16_3.9x4.9mm_P0.635mm
- removed U2: PCA9306DC1, Package_SO:VSSOP-8_2.3x2mm_P0.5mm
- removed U3: LD1117S18TR_SOT223, Package_TO_SOT_SMD:SOT-223-3_TabPin2
- removed U4: LD1117S25TR_SOT223, Package_TO_SOT_SMD:SOT-223-3_TabPin2
- removed U6: LD1117S12TR_SOT223, Package_TO_SOT_SMD:SOT-223-3_TabPin2
- removed U7: TCA9535DBR, Package_SO:SSOP-24_5.3x8.2mm_P0.65mm
- removed U8: TXB0104RUT, Package_DFN_QFN:Texas_R-PUQFN-N12
- added ?: , , F.Cu at (110.0, 91.0)
- added ?: , , F.Cu at (52.0, 91.0)
- added D6: LED, LED_SMD:LED_0402_1005Metric, F.Cu at (189.5, 124.5)
- added J3: Conn_02x30_Odd_Even, Connector_PinHeader_2.00mm:PinHeader_2x30_P2.00mm_Vertical_SMD, F.Cu at (82.0, 59.4)
- added J4: RJ45, Connector_RJ:RJ45_Amphenol_54602-x08_Horizontal, F.Cu at (120.0, 117.0)
- added J5: RJ45, Connector_RJ:RJ45_Amphenol_54602-x08_Horizontal, F.Cu at (145.0, 117.0)
- added J6: RJ45, Connector_RJ:RJ45_Amphenol_54602-x08_Horizontal, F.Cu at (170.0, 117.0)
- added J7: RJ45, Connector_RJ:RJ45_Amphenol_54602-x08_Horizontal, F.Cu at (195.0, 117.0)
- added J8: Barrel_Jack, spark:PJ1-021-SMT-TR, F.Cu at (30.0, 45.0)
- added LSI-U1: lsi-powermodule-7, lsi:lsi-powermodule-7, F.Cu at (133.0, 48.2)
- added P1: Conn_02x20_Odd_Even, spark:PinSocket_2x20_P2.54mm_Vertical_Inverted_SMD_Alignment_Pin, F.Cu at (81.0, 91.0)
- added R10: 4.7k, Resistor_SMD:R_0402_1005Metric, F.Cu at (157.0, 74.5)
- added R10: 4.7k, Resistor_SMD:R_0402_1005Metric, F.Cu at (189.9, 119.0)
- added R13: 1K, Resistor_SMD:R_0402_1005Metric, F.Cu at (159.9, 70.5)
- added R14: 1K, Resistor_SMD:R_0402_1005Metric, F.Cu at (159.9, 72.5)
- added R15: 1K, Resistor_SMD:R_0402_1005Metric, F.Cu at (159.9, 74.5)
- added R16: 1K, Resistor_SMD:R_0402_1005Metric, F.Cu at (162.8, 66.5)
- added R17: 1K, Resistor_SMD:R_0402_1005Metric, F.Cu at (162.8, 68.5)
- added R18: 1K, Resistor_SMD:R_0402_1005Metric, F.Cu at (162.8, 70.5)
- added R19: 4.7k, Resistor_SMD:R_0402_1005Metric, F.Cu at (64.9, 120.0)
- added R19: 4.7k, Resistor_SMD:R_0402_1005Metric, F.Cu at (162.8, 72.5)
- added R20: 4.7k, Resistor_SMD:R_0402_1005Metric, F.Cu at (162.8, 74.5)
- added R20: 4.7k, Resistor_SMD:R_0402_1005Metric, F.Cu at (64.9, 119.0)
- added R3: 4.7k, Resistor_SMD:R_0402_1005Metric, F.Cu at (154.1, 70.5)
- added R3: 4.7k, Resistor_SMD:R_0402_1005Metric, F.Cu at (114.9, 120.0)
- added R4: 4.7k, Resistor_SMD:R_0402_1005Metric, F.Cu at (114.9, 119.0)
- added R4: 4.7k, Resistor_SMD:R_0402_1005Metric, F.Cu at (154.1, 72.5)
- added R5: 4.7k, Resistor_SMD:R_0402_1005Metric, F.Cu at (139.9, 120.0)
- added R5: 4.7k, Resistor_SMD:R_0402_1005Metric, F.Cu at (154.1, 74.5)
- added R6: 4.7k, Resistor_SMD:R_0402_1005Metric, F.Cu at (139.9, 119.0)
- added R6: 4.7k, Resistor_SMD:R_0402_1005Metric, F.Cu at (157.0, 66.5)
- added R7: 4.7k, Resistor_SMD:R_0402_1005Metric, F.Cu at (157.0, 68.5)
- added R7: 4.7k, Resistor_SMD:R_0402_1005Metric, F.Cu at (164.9, 120.0)
- added R8: 4.7k, Resistor_SMD:R_0402_1005Metric, F.Cu at (164.9, 119.0)
- added R8: 4.7k, Resistor_SMD:R_0402_1005Metric, F.Cu at (157.0, 70.5)
- added R9: 4.7k, Resistor_SMD:R_0402_1005Metric, F.Cu at (157.0, 72.5)
- added R9: 4.7k, Resistor_SMD:R_0402_1005Metric, F.Cu at (189.9, 120.0)
- D1, D2, D3, D4, D5: value D_Schottky -> LED; footprint Diode_SMD:D_0402_1005Metric -> LED_SMD:LED_0402_1005Metric
- R1, R2: value 1k -> 4.7k
- moved U5 106.3 mm to (157.6, 79.7)
- moved D5 95.3 mm to (164.5, 125.0), turned to 0 degrees
- moved D4 76.2 mm to (139.5, 124.5), turned to 0 degrees
- moved D1 66.5 mm to (63.5, 123.5), turned to 0 degrees
- moved R1 65.3 mm to (90.0, 120.0)
- moved D3 63.2 mm to (114.0, 124.5), turned to 0 degrees
- moved D2 59.4 mm to (88.5, 124.0), turned to 0 degrees
- moved R2 57.5 mm to (90.0, 119.0), turned to 0 degrees
- moved J2 1.23 mm to (95.0, 117.0)
- moved J1 0.51 mm to (70.0, 117.0)
Connections:
- D1 pad 1: v_bus 1 -> LED_0
- D2 pad 1: v_bus 1 -> LED_1
- D3 pad 1: v_bus 1 -> LED_2
- D4 pad 1: v_bus 1 -> LED_3
- D5 pad 1: v_bus 1 -> LED_4
- J1 pad 2: Net-(U8-A1) -> unconnected-(J1-Pad2)
- J1 pad 3: Net-(U2-SCL1) -> SCL_0
- J1 pad 4: Net-(U8-A2) -> unconnected-(J1-Pad4)
- J1 pad 5: Net-(Q5-D) -> +3V3
- J1 pad 6: Net-(U8-A3) -> unconnected-(J1-Pad6)
- J1 pad 7: Net-(U2-SDA1) -> SDA_0
- J1 pad 8: bus 1 a 1 -> unconnected-(J1-Pad8)
- J2 pad 2: Net-(U8-A1) -> unconnected-(J2-Pad2)
- J2 pad 3: Net-(U2-SCL1) -> SCL_1
- J2 pad 4: Net-(U8-A2) -> unconnected-(J2-Pad4)
- J2 pad 5: Net-(Q6-D) -> +3V3
- J2 pad 6: Net-(U8-A3) -> unconnected-(J2-Pad6)
- J2 pad 7: Net-(U2-SDA1) -> SDA_1
- J2 pad 8: bus 1 a 2 -> unconnected-(J2-Pad8)
- P5 pad 10: unconnected-(P5-GPIO15/RXD-Pad10) -> GPIO15
- P5 pad 11: unconnected-(P5-GPIO17-Pad11) -> GPIO17
- P5 pad 12: unconnected-(P5-GPIO18/PWM0-Pad12) -> GPIO18
- P5 pad 13: CS_4 -> GPIO27
- P5 pad 14: unconnected-(P5-GND-Pad14) -> GND
- P5 pad 15: CS_5 -> GPIO22
- P5 pad 16: CS_2 -> GPIO23
- P5 pad 17: unconnected-(P5-3V3-Pad17) -> +3V3
- P5 pad 18: CS_3 -> unconnected-(P5-GPIO24-Pad18)
- P5 pad 20: unconnected-(P5-GND-Pad20) -> GND
- P5 pad 22: unconnected-(P5-GPIO25-Pad22) -> iCE_CDONE
- P5 pad 24: CS_0 -> iCE_SS_B
- P5 pad 25: unconnected-(P5-GND-Pad25) -> GND
- P5 pad 26: CS_1 -> GPIO7
- P5 pad 27: unconnected-(P5-ID_SD/GPIO0-Pad27) -> GPIO0
- P5 pad 28: unconnected-(P5-ID_SC/GPIO1-Pad28) -> GPIO1
- P5 pad 29: unconnected-(P5-GCLK1/GPIO5-Pad29) -> GPIO5
- P5 pad 3: SDA -> GPIO2
- P5 pad 30: unconnected-(P5-GND-Pad30) -> GND
- P5 pad 31: unconnected-(P5-GCLK2/GPIO6-Pad31) -> GPIO6
- P5 pad 32: unconnected-(P5-PWM0/GPIO12-Pad32) -> GPIO12
- P5 pad 33: unconnected-(P5-PWM1/GPIO13-Pad33) -> GPIO13
- P5 pad 34: unconnected-(P5-GND-Pad34) -> GND
- P5 pad 35: unconnected-(P5-GPIO19/MISO1-Pad35) -> GPIO19
- P5 pad 36: unconnected-(P5-GPIO16-Pad36) -> GPIO16
- P5 pad 37: unconnected-(P5-GPIO26-Pad37) -> GPIO26
- P5 pad 38: unconnected-(P5-GPIO20/MOSI1-Pad38) -> GPIO20
- P5 pad 39: unconnected-(P5-GND-Pad39) -> GND
- P5 pad 40: unconnected-(P5-GPIO21/SCLK1-Pad40) -> GPIO21
- P5 pad 5: SCL -> GPIO3
- P5 pad 6: unconnected-(P5-GND-Pad6) -> GND
- P5 pad 7: unconnected-(P5-GCLK0/GPIO4-Pad7) -> GPIO4
- P5 pad 8: unconnected-(P5-GPIO14/TXD-Pad8) -> GPIO14
- P5 pad 9: unconnected-(P5-GND-Pad9) -> GND
- R1 pad 1: bus 1  1.2v -> +3V3
- R1 pad 2: GND -> SDA_1
- R2 pad 1: GND -> +3V3
- R2 pad 2: bus 1  1.8v -> SCL_1
Routing:
- net SYS_DCIN: track 0.00 -> 110.3 mm
- net MOSI: track 107.5 -> 0.00 mm, vias 1 -> 0
- net MISO: track 105.9 -> 0.00 mm, vias 1 -> 0
- net SCK: track 104.7 -> 0.00 mm, vias 1 -> 0
- net bus 1 a 2: track 90.9 -> 0.00 mm, vias 1 -> 0
- net SDA 0: track 90.8 -> 0.00 mm, vias 4 -> 0
- net CS_1: track 86.7 -> 0.00 mm, vias 1 -> 0
- net SCL 0: track 86.2 -> 0.00 mm, vias 4 -> 0
- net v_bus 1: track 76.7 -> 0.00 mm, vias 6 -> 0
- net bus 1 a 1: track 66.5 -> 0.00 mm, vias 1 -> 0
- net CS_0: track 66.3 -> 0.00 mm
- net bus 1  5v: track 45.4 -> 0.00 mm, vias 2 -> 0
- net +1V8: track 44.2 -> 0.00 mm
- net +1V2: track 43.7 -> 0.00 mm
- net +2V5: track 42.5 -> 0.00 mm
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Other:
- board text added: "spark4pi-sensors-0.2"
- board text removed: "spark4pi-signals-0.1"
