File: board/spark.kicad_sch (KiCad schematic)
At the start: 77 parts, among them J1 RJ45, J2 RJ45, J3 RJ45, J4 RJ45, J5 RJ45, J6 RJ45, P5 Raspberry_Pi_2_3, Q1 IRLZ44N, Q10 IRLZ44N, Q11 IRLZ44N, Q12 IRLZ44N, Q13 IRLZ44N, Q14 IRLZ44N, Q15 IRLZ44N, Q16 IRLZ44N, Q17 IRLZ44N, Q18 IRLZ44N, Q19 IRLZ44N, Q2 IRLZ44N, Q20 IRLZ44N, Q21 IRLZ44N, Q3 IRLZ44N, Q4 IRLZ44N, Q5 IRLZ44N, Q6 IRLZ44N, Q7 IRLZ44N, Q8 IRLZ44N, Q9 IRLZ44N, U1 PCA9544APW, U10 TXB0104RUT, U11 MAX11614, U12 PCA9306DC1, U13 TXB0104RUT, U2 PCA9306DC1, U3 LD1117S18TR_SOT223, U4 LD1117S25TR_SOT223, U5 LD1117S33TR_SOT223, U6 LD1117S12TR_SOT223, U7 TCA9535DBR, U8 TXB0104RUT, U9 PCA9306DC1

Commit message: fix: added correct i2c busses
Connections:
- net SCL 0: no longer U12.6 (SCL2), U9.6 (SCL2)
- net SDA 0: no longer U12.5 (SDA2), U9.5 (SDA2)
- net SDA 2: now reaches U1.12 (SD2)
- net SDA 2: now also U12.5 (SDA2)
- net SCL 2: now reaches U1.13 (SC2)
- net SCL 2: now also U12.6 (SCL2)
- net SDA 1: now reaches U1.8 (SD1)
- net SDA 1: now also U9.5 (SDA2)
- net SCL 1: now reaches U1.9 (SC1)
- net SCL 1: now also U9.6 (SCL2)
Changed lines of the file:
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@@
+		)
+	)
+	(global_label "SCL 2"
+		(shape input)
+		(at 104.14 193.04 0)
+		(fields_autoplaced yes)
+		(effects
+			(font
+				(size 1.524 1.524)
+			)
+			(justify left)
+		)
+		(property "Intersheetrefs" "${INTERSHEET_REFS}"
+			(at 113.7584 193.04 0)
+			(effects
+				(font
+					(size 1.27 1.27)
+				)
+				(justify left)
+				(hide yes)
+			)
 		)
 	)
@@
 		)
 	)
-	(global_label "SCL 0"
+	(global_label "SCL 2"
 		(shape input)
 		(at 386.08 88.9 90)
@@
 		)
 	)
+	(global_label "SDA 2"
+		(shape input)
+		(at 104.14 190.5 0)
+		(fields_autoplaced yes)
+		(effects
+			(font
+				(size 1.524 1.524)
+			)
+			(justify left)
+		)
+		(property "Intersheetrefs" "${INTERSHEET_REFS}"
+			(at 113.831 190.5 0)
+			(effects
+				(font
+					(size 1.27 1.27)
+				)
+				(justify left)
+				(hide yes)
+			)
+		)
+	)
 	(global_label "CS_2"
 		(shape input)
@@
 		)
 	)
+	(global_label "SCL 1"
+		(shape input)
+		(at 104.14 182.88 0)
+		(fields_autoplaced yes)
+		(effects
+			(font
+				(size 1.524 1.524)
+			)
+			(justify left)
+		)
+		(property "Intersheetrefs" "${INTERSHEET_REFS}"
+			(at 113.7584 182.88 0)
+			(effects
+				(font
+					(size 1.27 1.27)
+				)
+				(justify left)
+				(hide yes)
+			)
+		)
+	)
 	(global_label "v_bus 3"
 		(shape input)
@@
 		)
 	)
+	(global_label "SDA 1"
+		(shape input)
+		(at 104.14 180.34 0)
+		(fields_autoplaced yes)
+		(effects
+			(font
+				(size 1.524 1.524)
+			)
+			(justify left)
+		)
+		(property "Intersheetrefs" "${INTERSHEET_REFS}"
+			(at 113.831 180.34 0)
+			(effects
+				(font
+					(size 1.27 1.27)
+				)
+				(justify left)
+				(hide yes)
+			)
+		)
+	)
 	(global_label "bus 2  5v"
 		(shape input)
@@
 		)
 	)
-	(global_label "SDA 0"
+	(global_label "SDA 1"
 		(shape input)
 		(at 237.49 87.63 90)
@@
 		)
 	)
-	(global_label "SCL 0"
+	(global_label "SCL 1"
 		(shape input)
 		(at 234.95 87.63 90)
@@
 		)
 	)
-	(global_label "SDA 0"
+	(global_label "SDA 2"
 		(shape input)
 		(at 388.62 88.9 90)

Commit message: feat: added pull ups
Parts:
- added D16: Active LED, LED_SMD:LED_0402_1005Metric, symbol Device:LED
- added R22, R23, R24, R25, R26, R27, R28, R29, R30, R31, R32, R33: 4.7k, Resistor_SMD:R_0402_1005Metric, symbol Device:R
Connections:
- net +5V: now also R22.1, R23.1, R24.1, R25.1, R26.1, R27.1, R28.1, R29.1, R30.1, R31.1
- net CS_0: now also D16.2 (A); no longer Q6.1 (G), R6.2
- net SCL: now also R23.2
- net SCL 0: now also R30.2
- net SCL 1: now also R28.2
- net SCL 2: now also R26.2
- net SCL 3: now also R24.2
- net SDA: now also R22.2
- net SDA 0: now also R31.2
- net SDA 1: now also R29.2
- net SDA 2: now also R27.2
- net SDA 3: now also R25.2
- net at J1.3, J2.3, U2.3 (SCL1): now also R33.2
- net at J1.7, J2.7, U2.4 (SDA1): now also R32.2
- net at J1.5, Q6.2 (D): now also R32.1, R33.1
- new net: D16.1 (K), Q6.1 (G), R6.2
Other:
- title: spark4pi-digital-io-2.10 -> spark4pi-sensors-0.01
- moved on the sheet: D10, D11, D12, D13, D14, D15, D6, D7, D8, D9, J2, J3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

Commit message: feat: initial board stuff
Parts:
- removed Q1, Q2, Q3, Q4, Q5, Q6, Q7: IRLZ44N, Package_TO_SOT_THT:TO-220-3_Vertical, symbol Transistor_FET:IRLZ44N
- added D17: Active LED, LED_SMD:LED_0402_1005Metric, symbol Device:LED
- added Q1, Q2, Q22, Q3, Q4, Q5, Q6: AO3400A, Package_TO_SOT_SMD:SOT-23, symbol Transistor_FET:AO3400A
- R1, R2, R3, R4, R5, R6, R7: footprint Resistor_SMD:R_01005_0402Metric -> Resistor_SMD:R_0402_1005Metric
Connections:
- net +1V2: now also Q22.2 (S)
- net +1V8: now also Q1.2 (S)
- net +2V5: now also Q2.2 (S)
- net +3V3: now also Q3.2 (S)
- net +5V: now also Q4.2 (S)
- net CS_0: no longer R7.2
- net CS_1: now also D17.2 (A)
- net GND: now also R1.2; no longer R1.1
- net bus 1  1.2v: now also R1.1, Q22.1 (G); no longer R1.2
- net bus 1  1.8v: now also Q1.1 (G)
- net bus 1  2.5v: now also Q2.1 (G)
- net bus 1  3.3v: now also Q3.1 (G)
- net bus 1  5v: now also Q4.1 (G)
- net v_bus 1: now also Q5.2 (S), Q6.2 (S)
- net at J2.5: now also Q6.3 (D)
- net at D16.1 (K), R6.2: now also Q5.1 (G)
- net at D2.2 (A): now also Q1.3 (D)
- net at J1.5, R32.1, R33.1: now also Q5.3 (D)
- net at D4.2 (A): now also Q3.3 (D)
- net at D1.2 (A): now also Q22.3 (D)
- net at D3.2 (A): now also Q2.3 (D)
- net at D5.2 (A): now also Q4.3 (D)
- new net: D17.1 (K), Q6.1 (G), R7.2
Other:
- moved on the sheet: R1

Commit message: feat: inital version
Connections:
- net +3V3: now also P5.17 (3V3)
- net GND: now also P5.14 (GND), P5.20 (GND), P5.25 (GND), P5.30 (GND), P5.34 (GND), P5.39 (GND), P5.6 (GND), P5.9 (GND)
- net bus 1  1.2v: now also U7.8 (P04); no longer U7.4 (P00)
- net bus 1  1.8v: now also U7.7 (P03); no longer U7.5 (P01)
- net bus 1  3.3v: now also U7.5 (P01); no longer U7.7 (P03)
- net bus 1  5v: now also U7.4 (P00); no longer U7.8 (P04)

Commit message: feat: rev 2
Parts:
- removed D1, D10, D11, D12, D13, D14, D15, D2, D3, D4, D5, D6, D7, D8, D9: D_Schottky, Diode_SMD:D_0402_1005Metric, symbol Device:D_Schottky
- removed D16, D17: Active LED, LED_SMD:LED_0402_1005Metric, symbol Device:LED
- removed J3: RJ45, Connector_RJ:RJ45_Amphenol_54602-x08_Horizontal, symbol Connector:RJ45
- removed Q1, Q2, Q22, Q3, Q4, Q5, Q6: AO3400A, Package_TO_SOT_SMD:SOT-23, symbol Transistor_FET:AO3400A
- removed Q10, Q11, Q12, Q13, Q14, Q15, Q16, Q17, Q18, Q19, Q20, Q21, Q8, Q9: IRLZ44N, Package_TO_SOT_THT:TO-220-3_Vertical, symbol Transistor_FET:IRLZ44N
- removed R11, R12, R19, R20, R21: 1k, Resistor_SMD:R_01005_0402Metric, symbol Device:R
- removed R24, R25, R26, R27, R28, R29, R30, R31, R32, R33: 4.7k, Resistor_SMD:R_0402_1005Metric, symbol Device:R
- removed U1: PCA9544APW, Package_SO:TSSOP-20_4.4x6.5mm_P0.65mm, symbol Interface_Expansion:PCA9544APW
- removed U10, U13, U8: TXB0104RUT, Package_DFN_QFN:Texas_R-PUQFN-N12, symbol Logic_LevelTranslator:TXB0104RUT
- removed U11: MAX11614, Package_SO:QSOP-16_3.9x4.9mm_P0.635mm, symbol Analog_ADC:MAX11614
- removed U12, U2, U9: PCA9306DC1, Package_SO:VSSOP-8_2.3x2mm_P0.5mm, symbol Interface:PCA9306DC1
- removed U3: LD1117S18TR_SOT223, Package_TO_SOT_SMD:SOT-223-3_TabPin2, symbol Regulator_Linear:LD1117S18TR_SOT223
- removed U4: LD1117S25TR_SOT223, Package_TO_SOT_SMD:SOT-223-3_TabPin2, symbol Regulator_Linear:LD1117S25TR_SOT223
- removed U6: LD1117S12TR_SOT223, Package_TO_SOT_SMD:SOT-223-3_TabPin2, symbol Regulator_Linear:LD1117S12TR_SOT223
- removed U7: TCA9535DBR, Package_SO:SSOP-24_5.3x8.2mm_P0.65mm, symbol Interface_Expansion:TCA9535DBR
- added D1, D2, D3, D4, D5, D6: LED, LED_SMD:LED_0402_1005Metric, symbol Device:LED
- added J3: Conn_02x30_Odd_Even, Connector_PinHeader_2.00mm:PinHeader_2x30_P2.00mm_Vertical_SMD, symbol Connector_Generic:Conn_02x30_Odd_Even
- added J7: RJ45, Connector_RJ:RJ45_Amphenol_54602-x08_Horizontal, symbol Connector:RJ45
- added J8: Barrel_Jack, spark:PJ1-021-SMT-TR, symbol Connector:Barrel_Jack_Switch
- added LSI-U1: lsi-powermodule-7, lsi:lsi-powermodule-7, symbol lsi:lsi-powermodule-7
- added P1: Conn_02x20_Odd_Even, spark:PinSocket_2x20_P2.54mm_Vertical_Inverted_SMD_Alignment_Pin, symbol Connector_Generic:Conn_02x20_Odd_Even
- R1, R2, R3, R4, R5, R6, R7: value 1k -> 4.7k
- R10, R8, R9: value 1k -> 4.7k; footprint Resistor_SMD:R_01005_0402Metric -> Resistor_SMD:R_0402_1005Metric
- R13, R14, R15, R16, R17, R18: value 1k -> 1K; footprint Resistor_SMD:R_01005_0402Metric -> Resistor_SMD:R_0402_1005Metric
- renumbered R22 to R19, R23 to R20
Connections:
- net bus 1  1.2v is gone; now on net +3V3: R1.1
- net bus 1  2.5v is gone; now on net SDA_2: R3.2
- net bus 1  3.3v is gone; now on net SCL_2: R4.2
- net bus 1  5v is gone; now on net SDA_3: R5.2
- net +3V3: now also J1.5, J2.5, J4.5, J5.5, J6.5, R10.1, R13.1, R14.1, R15.1, R16.1, R17.1, R18.1, R19.1, R2.1, R20.1, R3.1, R4.1, R5.1, R6.1, R7.1, R8.1, R9.1, J7.5, P1.1 (Pin_1), P1.17 (Pin_17)
- net +5V: now also LSI-U1.3 (VPP_OUT), P1.2 (Pin_2), P1.4 (Pin_4); no longer R19.1, R20.1
- net GND: now also J7.1, J8.2, J8.3, LSI-U1.1 (GND), LSI-U1.4 (GND), P1.14 (Pin_14), P1.20 (Pin_20), P1.25 (Pin_25), P1.30 (Pin_30), P1.34 (Pin_34), P1.39 (Pin_39), P1.6 (Pin_6), P1.9 (Pin_9); no longer R1.2, R10.1, R13.1, R14.1, R15.1, R16.1, R17.1, R18.1, R2.1, R3.1, R4.1, R5.1, R6.1, R7.1, R8.1, R9.1
- net MISO: now also P1.21 (Pin_21)
- net MOSI: now also P1.19 (Pin_19)
- net SCK: now also P1.23 (Pin_23)
- net GPIO15: now reaches P5.10 (GPIO15/RXD)
- net GPIO15: now also P1.10 (Pin_10)
- net GPIO17: now reaches P5.11 (GPIO17)
- net GPIO17: now also P1.11 (Pin_11)
- net GPIO18: now reaches P5.12 (GPIO18/PWM0)
- net GPIO18: now also P1.12 (Pin_12)
- net iCE_CDONE: now reaches P5.22 (GPIO25)
- net iCE_CDONE: now also P1.22 (Pin_22)
- net GPIO0: now reaches P5.27 (ID_SD/GPIO0)
- net GPIO0: now also P1.27 (Pin_27)
- net GPIO1: now reaches P5.28 (ID_SC/GPIO1)
- net GPIO1: now also P1.28 (Pin_28)
- net GPIO5: now reaches P5.29 (GCLK1/GPIO5)
- net GPIO5: now also P1.29 (Pin_29)
- net GPIO6: now reaches P5.31 (GCLK2/GPIO6)
- net GPIO6: now also P1.31 (Pin_31)
- net GPIO12: now reaches P5.32 (PWM0/GPIO12)
- net GPIO12: now also P1.32 (Pin_32)
- net GPIO13: now reaches P5.33 (PWM1/GPIO13)
- net GPIO13: now also P1.33 (Pin_33)
- net GPIO19: now reaches P5.35 (GPIO19/MISO1)
- net GPIO19: now also P1.35 (Pin_35)
- net GPIO16: now reaches P5.36 (GPIO16)
- net GPIO16: now also P1.36 (Pin_36)
- net GPIO26: now reaches P5.37 (GPIO26)
- net GPIO26: now also P1.37 (Pin_37)
- net GPIO20: now reaches P5.38 (GPIO20/MOSI1)
- net GPIO20: now also P1.38 (Pin_38)
- net GPIO21: now reaches P5.40 (GPIO21/SCLK1)
- net GPIO21: now also P1.40 (Pin_40)
- net GPIO4: now reaches P5.7 (GCLK0/GPIO4)
- net GPIO4: now also P1.7 (Pin_7)
- net GPIO14: now reaches P5.8 (GPIO14/TXD)
- net GPIO14: now also P1.8 (Pin_8)
- net SCL_3: now reaches J5.3
- net SCL_3: now also R6.2, J3.15 (Pin_15); no longer J6.3
- net SDA_3: now reaches J5.7
- net SDA_3: now also J3.13 (Pin_13); no longer J6.7
- net at J2.2: no longer J1.2
- net SCL_0: now reaches J1.3
- net SCL_0: now also R20.2, J3.3 (Pin_3); no longer J2.3
- net at J2.4: no longer J1.4
- net at J2.6: no longer J1.6
- net SDA_0: now reaches J1.7
- net SDA_0: now also R19.2, J3.1 (Pin_1); no longer J2.7
- net SDA_4: now reaches R7.2
- net SDA_4: now also J6.7, J3.17 (Pin_17)
- net SCL_2: now reaches J4.3
- net SCL_2: now also J3.11 (Pin_11)
- net SDA_2: now reaches J4.7
- net SDA_2: now also J3.9 (Pin_9)
- net at J5.2: no longer J6.2
- net at J5.4: no longer J6.4
- net at J5.6: no longer J6.6
- net CS_0 renamed iCE_SS_B
- net iCE_SS_B: now also P1.24 (Pin_24)
- net CS_1 renamed GPIO7
- net GPIO7: now also P1.26 (Pin_26)
- net CS_2 renamed GPIO23
- net GPIO23: now also P1.16 (Pin_16)
- net CS_3: no longer names the net of P5.18 (GPIO24)
- net CS_3: no longer R14.2
- net CS_4: no longer names the net of R18.2
- net CS_4: now also D6.2 (A); no longer P5.13 (GPIO27)
- net CS_5 renamed GPIO22
- net GPIO22: now also P1.15 (Pin_15)
- net SCL renamed GPIO3
- net GPIO3: now also P1.5 (Pin_5); no longer R20.2
- net SDA renamed GPIO2
- net GPIO2: now also P1.3 (Pin_3); no longer R19.2
- net bus 1  1.8v renamed SCL_1
- net SCL_1: now also J2.3, J3.7 (Pin_7)
- net bus 1 a 1: no longer names the net of J1.8
- net bus 1 a 2: no longer names the net of J2.8
- net bus 2  1.2v renamed SCL_4
- net SCL_4: now also J6.3, J3.19 (Pin_19)
- net bus 2  1.8v renamed SDA_5
- net SDA_5: now also J3.21 (Pin_21), J7.7
- net bus 2  3.3v: no longer names the net of R13.2
- net bus 2  3.3v: now also D1.2 (A)
- net bus 2  5v renamed SCL_5
- net SCL_5: now also J3.23 (Pin_23), J7.3
- net bus 2 a 2: no longer names the net of J4.8
- net bus 3  1.2v: no longer names the net of R15.2
- net bus 3  1.2v: now also D3.2 (A)
- net bus 3  1.8v: no longer names the net of R16.2
- net bus 3  1.8v: now also D4.2 (A)
- net bus 3  5v: no longer names the net of R17.2
- net bus 3  5v: now also D5.2 (A)
- net bus 3 a 1: no longer names the net of J5.8
- net bus 3 a 2: no longer names the net of J6.8
- new net: D2.2 (A), R14.2
- new net GPIO27: P1.13 (Pin_13), P5.13 (GPIO27)
- new net LED_0: D1.1 (K), J3.2 (Pin_2)
- new net LED_1: D2.1 (K), J3.4 (Pin_4)
- new net LED_2: D3.1 (K), J3.6 (Pin_6)
- new net LED_3: D4.1 (K), J3.8 (Pin_8)
- new net LED_4: D5.1 (K), J3.10 (Pin_10)
- new net LED_5: D6.1 (K), J3.12 (Pin_12)
- new net SCL_6: J3.27 (Pin_27)
- new net SDA_1: J2.7, J3.5 (Pin_5), R1.2
- new net SDA_6: J3.25 (Pin_25)
- new net SYS_DCIN: J8.1, LSI-U1.2 (VPP_IN)
- new net iCE_CREST: P1.18 (Pin_18)
- no-connect marks 0 -> 4
Other:
- note removed: "1.2"
- note removed: "1.8"
- note removed: "2.5"
- title: spark4pi-sensors-0.01 -> spark4pi-sensors-0.02
- moved on the sheet: J1, P5, R19, R20, U5
